Commit message: First stable version

File: robotiq_85_description/urdf/robotiq_85_gripper.transmission.xacro (robot description, xacro)
@@ -5,30 +5,73 @@
             <type>transmission_interface/SimpleTransmission</type>
             <joint name="${prefix}gripper_finger1_joint">
-                <hardwareInterface>PositionJointInterface</hardwareInterface>
+                <hardwareInterface>hardware_interface/EffortJointInterface</hardwareInterface>
             </joint>
             <actuator name="${prefix}gripper_finger1_motor">
                 <mechanicalReduction>1</mechanicalReduction>
-                <hardwareInterface>PositionJointInterface</hardwareInterface>
+                <hardwareInterface>hardware_interface/EffortJointInterface</hardwareInterface>
             </actuator>
         </transmission>
-        <gazebo>
-                <!-- loading plugin: mimic joints works in gazebo now -->
+        <transmission name="${prefix}gripper_finger2_trans">
+            <type>transmission_interface/SimpleTransmission</type>
+            <joint name="${prefix}gripper_finger2_joint">
+                <hardwareInterface>hardware_interface/EffortJointInterface</hardwareInterface>
+            </joint>
+            <actuator name="${prefix}gripper_finger2_motor">
+                <mechanicalReduction>1</mechanicalReduction>
+                <hardwareInterface>hardware_interface/EffortJointInterface</hardwareInterface>
+            </actuator>
+        </transmission>
+        <transmission name="gripper_finger2_inner_knuckle_trans">
+            <type>transmission_interface/SimpleTransmission</type>
+            <joint name="gripper_finger2_inner_knuckle_joint">
+                <hardwareInterface>hardware_interface/EffortJointInterface</hardwareInterface>
+            </joint>
+            <actuator name="gripper_finger2_inner_knuckle_motor">
+                <mechanicalReduction>1</mechanicalReduction>
+                <hardwareInterface>hardware_interface/EffortJointInterface</hardwareInterface>
+            </actuator>
+        </transmission>
+        <transmission name="gripper_finger1_inner_knuckle_trans">
+            <type>transmission_interface/SimpleTransmission</type>
+            <joint name="gripper_finger1_inner_knuckle_joint">
+                <hardwareInterface>hardware_interface/EffortJointInterface</hardwareInterface>
+            </joint>
+            <actuator name="gripper_finger1_inner_knuckle_motor">
+                <mechanicalReduction>1</mechanicalReduction>
+                <hardwareInterface>hardware_interface/EffortJointInterface</hardwareInterface>
+            </actuator>
+        </transmission>
+        <transmission name="${prefix}gripper_finger1_finger_tip_trans">
+            <type>transmission_interface/SimpleTransmission</type>
+            <joint name="${prefix}gripper_finger1_finger_tip_joint">
+                <hardwareInterface>hardware_interface/EffortJointInterface</hardwareInterface>
+            </joint>
+            <actuator name="${prefix}gripper_finger1_finger_tip_motor">
+                <mechanicalReduction>1</mechanicalReduction>
+                <hardwareInterface>hardware_interface/EffortJointInterface</hardwareInterface>
+            </actuator>
+        </transmission>
+        <transmission name="${prefix}gripper_finger2_finger_tip_trans">
+            <type>transmission_interface/SimpleTransmission</type>
+            <joint name="${prefix}gripper_finger2_finger_tip_joint">
+                <hardwareInterface>hardware_interface/EffortJointInterface</hardwareInterface>
+            </joint>
+            <actuator name="${prefix}gripper_finger2_finger_tip_motor">
+                <mechanicalReduction>1</mechanicalReduction>
+                <hardwareInterface>hardware_interface/EffortJointInterface</hardwareInterface>
+            </actuator>
+        </transmission>
+        <!--<gazebo>
             <plugin filename="libroboticsgroup_gazebo_mimic_joint_plugin.so" name="${prefix}mimic_robotiq_85_1">
                 <joint>${prefix}gripper_finger1_joint</joint>
                 <mimicJoint>${prefix}gripper_finger2_joint</mimicJoint>
-                <!--multiplier>1.0</multiplier>
-                <offset>0.0</offset-->
             </plugin>
             <plugin filename="libroboticsgroup_gazebo_mimic_joint_plugin.so" name="${prefix}mimic_robotiq_85_2">
                 <joint>${prefix}gripper_finger1_joint</joint>
                 <mimicJoint>${prefix}gripper_finger2_inner_knuckle_joint</mimicJoint>
-                <!--multiplier>1.0</multiplier>
-                <offset>0.0</offset-->
             </plugin>
             <plugin filename="libroboticsgroup_gazebo_mimic_joint_plugin.so" name="${prefix}mimic_robotiq_85_3">
                 <joint>${prefix}gripper_finger1_joint</joint>
                 <mimicJoint>${prefix}gripper_finger1_inner_knuckle_joint</mimicJoint>
-                <!--multiplier>1.0</multiplier>
-                <offset>0.0</offset-->
             </plugin>
             <plugin filename="libroboticsgroup_gazebo_mimic_joint_plugin.so" name="${prefix}mimic_robotiq_85_4">
@@ -44,4 +87,21 @@
                 <offset>0.0</offset>
             </plugin>
+        </gazebo>-->
+        <gazebo>
+            <plugin name="gazebo_grasp_fix" filename="libgazebo_grasp_fix.so">
+                <arm>
+                    <arm_name>ur10</arm_name>
+                    <palm_link>ur10_arm_wrist_3_link</palm_link>
+                    <gripper_link>gripper_finger1_finger_tip_link</gripper_link>
+                    <gripper_link>gripper_finger2_finger_tip_link</gripper_link>
+                </arm>
+                <forces_angle_tolerance>100</forces_angle_tolerance>
+                <update_rate>10</update_rate>
+                <grip_count_threshold>1</grip_count_threshold>
+                <max_grip_count>8</max_grip_count>
+                <release_tolerance>0.01</release_tolerance>
+                <disable_collisions_on_attach>false</disable_collisions_on_attach>
+                <contact_topic>__default_topic__</contact_topic>
+            </plugin>
         </gazebo>
     </xacro:macro>

File: robotiq_85_description/urdf/robotiq_85_gripper.urdf.xacro (robot description, xacro)
@@ -46,6 +46,6 @@
             <axis xyz="0 0 1"/>
             <origin rpy="0.0 0.0 0.0" xyz="0.05490451627 -0.03060114443 0.0"/>
-            <limit lower="-3.14" upper="3.14" velocity="100.0" effort="1000"/>
-            <mimic joint="${prefix}gripper_finger1_joint"/>
+            <limit lower="0.0" upper="0.804" velocity="2.0" effort="1000"/>
+            <mimic joint="${prefix}gripper_finger1_joint" offset="0"/>
         </joint>
         <link name="${prefix}gripper_finger1_knuckle_link">
@@ -105,4 +105,6 @@
             <child link="${prefix}gripper_finger1_finger_link"/>
             <origin xyz="-0.00408552455 -0.03148604435 0.0" rpy="0 0 0" />
+            <axis xyz="0 0 1"/>
+            <limit lower="0.0" upper="0.804" velocity="2.0" effort="1000"/>
         </joint>
         <joint name="${prefix}gripper_finger2_finger_joint" type="fixed">
@@ -110,4 +112,6 @@
             <child link="${prefix}gripper_finger2_finger_link"/>
             <origin xyz="-0.00408552455 -0.03148604435 0.0" rpy="0 0 0" />
+            <axis xyz="0 0 1"/>
+            <limit lower="0.0" upper="0.804" velocity="2.0" effort="1000"/>
         </joint>
         <link name="${prefix}gripper_finger1_finger_link">
@@ -168,5 +172,5 @@
             <axis xyz="0 0 1"/>
             <origin xyz="0.06142 0.0127 0" rpy="${pi} 0.0 0.0" />
-            <limit lower="-3.14" upper="3.14" velocity="100.0" effort="0.1"/>
+            <limit lower="0.0" upper="0.804" velocity="2.0" effort="1000"/>
             <mimic joint="${prefix}gripper_finger1_joint" offset="0"/>
         </joint>
@@ -176,5 +180,5 @@
             <axis xyz="0 0 1"/>
             <origin xyz="0.06142 -0.0127 0" rpy="0 0 0"/>
-            <limit lower="-3.14" upper="3.14" velocity="100.0" effort="0.1"/>
+            <limit lower="0.0" upper="0.804" velocity="2.0" effort="1000"/>
             <mimic joint="${prefix}gripper_finger1_joint" offset="0"/>
         </joint>
@@ -236,5 +240,5 @@
             <axis xyz="0 0 1"/>
             <origin xyz="0.04303959807 -0.03759940821 0.0" rpy="0.0 0.0 0.0"/>
-            <limit lower="-3.14" upper="3.14" velocity="100.0" effort="0.1"/>
+            <limit lower="-0.804" upper="0.0" velocity="2.0" effort="1000"/>
             <mimic joint="${prefix}gripper_finger1_joint" multiplier="-1"/>
         </joint>
@@ -244,5 +248,5 @@
             <axis xyz="0 0 1"/>
             <origin rpy="0.0 0.0 0.0" xyz="0.04303959807 -0.03759940821  0.0"/>
-            <limit lower="-3.14" upper="3.14" velocity="100.0" effort="0.1"/>
+            <limit lower="-0.804" upper="0.0" velocity="2.0" effort="1000"/>
             <mimic joint="${prefix}gripper_finger1_joint" multiplier="-1"/>
         </joint>
@@ -267,9 +271,9 @@
         </link>
         <gazebo reference="${prefix}gripper_finger1_finger_tip_link">
-            <implicitSpringDamper>1</implicitSpringDamper>
-            <mu1>100000</mu1>
-            <mu2>100000</mu2>
-            <kp>100000000.0</kp>
-            <kd>1.0</kd>
+            <mu1>100000</mu1>
+            <mu2>100000</mu2>
+            <kp>100000000.0</kp>
+            <kd>1.0</kd>
+            <fdir1>0 0 1</fdir1>
         </gazebo>
         <link name="${prefix}gripper_finger2_finger_tip_link">
@@ -293,9 +297,9 @@
         </link>
         <gazebo reference="${prefix}gripper_finger2_finger_tip_link">
-            <implicitSpringDamper>1</implicitSpringDamper>
-            <mu1>100000</mu1>
-            <mu2>100000</mu2>
-            <kp>100000000.0</kp>
-            <kd>1.0</kd>
+            <mu1>100000</mu1>
+            <mu2>100000</mu2>
+            <kp>100000000.0</kp>
+            <kd>1.0</kd>
+            <fdir1>0 0 1</fdir1>
         </gazebo>
         <xacro:robotiq_85_gripper_transmission prefix="${prefix}" />
